File: 02_PCB/Fast_SiPM_Photodetector/HVPowerSupply.kicad_sch (KiCad schematic)
At the start: 18 parts, among them IC1 LT8365JMSE

Commit message: feat(detector): update schematic and pcb after first prototype
Parts:
- D2: value SMD115PBQ-TP -> RB021VAM90TR
Connections:
- net EN renamed HV_EN
- net FBX renamed HV_FB
Other:
- note added: "HV Power Supply"
- moved on the sheet: C1
Changed lines of the file:
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@@
+		)
+	)
+	(text "HV Power Supply"
+		(exclude_from_sim no)
+		(at 152.4 35.814 0)
+		(effects
+			(font
+				(size 3.81 3.81)
+				(thickness 0.508)
+				(bold yes)
+			)
 		)
 	)
@@
 	)
 	(junction
-		(at 53.34 101.6)
-		(diameter 0)
-		(color 0 0 0 0)
-	)
-	(junction
-		(at 53.34 86.36)
+		(at 54.61 86.36)
 		(diameter 0)
 		(color 0 0 0 0)
@@
 	(wire
 		(pts
-			(xy 53.34 101.6) (xy 73.66 101.6)
+			(xy 54.61 101.6) (xy 73.66 101.6)
 		)
 		(stroke
@@
 	(wire
 		(pts
-			(xy 53.34 86.36) (xy 60.96 86.36)
+			(xy 54.61 86.36) (xy 60.96 86.36)
 		)
 		(stroke
@@
 	(wire
 		(pts
-			(xy 53.34 97.79) (xy 53.34 101.6)
+			(xy 54.61 97.79) (xy 54.61 101.6)
 		)
 		(stroke
@@
 	(wire
 		(pts
-			(xy 48.26 86.36) (xy 53.34 86.36)
+			(xy 49.53 86.36) (xy 54.61 86.36)
 		)
 		(stroke
@@
 	(wire
 		(pts
-			(xy 266.7 132.08) (xy 271.78 132.08)
+			(xy 266.7 132.08) (xy 275.59 132.08)
 		)
 		(stroke
@@
 	(wire
 		(pts
-			(xy 48.26 101.6) (xy 53.34 101.6)
-		)
-		(stroke
-			(width 0)
-			(type default)
-		)
-	)
-	(wire
-		(pts
-			(xy 53.34 86.36) (xy 53.34 90.17)
+			(xy 54.61 86.36) (xy 54.61 90.17)
 		)
 		(stroke
@@
 		)
 	)
-	(label "EN"
+	(label "HV_EN"
 		(at 120.65 97.79 0)
 		(effects
@@
 		)
 	)
-	(label "EN"
-		(at 271.78 132.08 180)
+	(label "HV_EN"
+		(at 275.59 132.08 180)
 		(effects
 			(font
@@
 		)
 	)
-	(label "FBX"
+	(label "HV_FB"
 		(at 120.65 113.03 0)
 		(effects
@@
 		)
 	)
-	(label "FBX"
-		(at 274.32 72.39 0)
+	(label "HV_FB"
+		(at 274.32 72.39 180)
 		(effects
 			(font
 				(size 1.27 1.27)
 			)
-			(justify left bottom)
-		)
-	)
-	(hierarchical_label "GND"
-		(shape input)
-		(at 48.26 101.6 180)
-		(effects
-			(font
-				(size 1.27 1.27)
-			)
-			(justify right)
+			(justify right bottom)
 		)
 	)
 	(hierarchical_label "VIN"
 		(shape input)
-		(at 48.26 86.36 180)
+		(at 49.53 86.36 180)
 		(effects
 			(font
@@
 			)
 		)
-		(property "Value" "SMD115PBQ-TP"
+		(property "Value" "RB021VAM90TR"
 			(at 197.104 83.058 0)
 			(show_name no)
@@
 	(symbol
 		(lib_id "Device:C")
-		(at 53.34 93.98 180)
+		(at 54.61 93.98 180)
 		(unit 1)
 		(body_style 1)
@@
 		(dnp no)
 		(property "Reference" "C1"
-			(at 56.642 92.71 0)
+			(at 57.912 92.71 0)
 			(show_name no)
 			(do_not_autoplace no)
@@
 		)
 		(property "Value" "10u;50V"
-			(at 56.642 95.25 0)
+			(at 57.912 95.25 0)
 			(show_name no)
 			(do_not_autoplace no)
@@
 		)
 		(property "Footprint" "Capacitor_SMD:C_1206_3216Metric"
-			(at 52.3748 90.17 0)
+			(at 53.6448 90.17 0)
 			(hide yes)
 			(show_name no)
@@
 		)
 		(property "Datasheet" ""
-			(at 53.34 93.98 0)
+			(at 54.61 93.98 0)
 			(hide yes)
 			(show_name no)
@@
 		)
 		(property "Description" "Unpolarized capacitor"
-			(at 53.34 93.98 0)
-			(hide yes)
-			(show_name no)
+			(at 54.61 93.98 0)
+			(hide yes)
+			(show_name no)
