File: 02_PCB/Fast_SiPM_Photodetector/InputProtection.kicad_sch (KiCad schematic)
At the start: 5 parts, among them Q1 PJA3463_R1_00001, SW1 JS202011JAQN

Commit message: feat(detector): update schematic and pcb after first prototype
Parts:
- SW1: value JS202011JAQN -> JS202011JCQN
Other:
- note added: "Input Protection"
- note removed: "Check Q1 pinout in final design!"
Changed lines of the file:
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@@
 		(title "Fast SiPM Photodetector")
 	)
-	(text "Check Q1 pinout in final design!"
+	(text "Input Protection"
 		(exclude_from_sim no)
-		(at 127.762 75.692 0)
+		(at 144.018 36.322 0)
 		(effects
 			(font
-				(size 1.27 1.27)
-			)
-		)
+				(size 3.81 3.81)
+				(thickness 0.508)
+				(bold yes)
+			)
+		)
+	)
+	(junction
+		(at 157.48 111.76)
+		(diameter 0)
+		(color 0 0 0 0)
 	)
 	(junction
@@
 	)
 	(junction
-		(at 157.48 123.19)
-		(diameter 0)
-		(color 0 0 0 0)
-	)
-	(junction
 		(at 137.16 88.9)
 		(diameter 0)
@@
 		(color 0 0 0 0)
 	)
-	(junction
-		(at 127 123.19)
-		(diameter 0)
-		(color 0 0 0 0)
-	)
 	(no_connect
 		(at 170.18 91.44)
@@
 	(wire
 		(pts
-			(xy 127 123.19) (xy 172.72 123.19)
+			(xy 157.48 111.76) (xy 157.48 115.57)
 		)
 		(stroke
@@
 	(wire
 		(pts
-			(xy 172.72 96.52) (xy 172.72 123.19)
+			(xy 172.72 96.52) (xy 172.72 111.76)
 		)
 		(stroke
@@
 	(wire
 		(pts
+			(xy 157.48 111.76) (xy 172.72 111.76)
+		)
+		(stroke
+			(width 0)
+			(type default)
+		)
+	)
+	(wire
+		(pts
 			(xy 127 96.52) (xy 127 99.06)
 		)
@@
 	(wire
 		(pts
-			(xy 88.9 123.19) (xy 127 123.19)
-		)
-		(stroke
-			(width 0)
-			(type default)
-		)
-	)
-	(wire
-		(pts
-			(xy 127 110.49) (xy 127 123.19)
-		)
-		(stroke
-			(width 0)
-			(type default)
-		)
-	)
-	(wire
-		(pts
-			(xy 157.48 99.06) (xy 157.48 123.19)
+			(xy 127 110.49) (xy 127 115.57)
+		)
+		(stroke
+			(width 0)
+			(type default)
+		)
+	)
+	(wire
+		(pts
+			(xy 157.48 99.06) (xy 157.48 111.76)
 		)
 		(stroke
@@
 			(width 0)
 			(type default)
-		)
-	)
-	(hierarchical_label "GND"
-		(shape input)
-		(at 88.9 123.19 180)
-		(effects
-			(font
-				(size 1.27 1.27)
-			)
-			(justify right)
 		)
 	)
@@
 			)
 			(justify right)
+		)
+	)
+	(symbol
+		(lib_id "power:GND")
+		(at 127 115.57 0)
+		(unit 1)
+		(body_style 1)
+		(exclude_from_sim no)
+		(in_bom yes)
+		(on_board yes)
+		(in_pos_files yes)
+		(dnp no)
+		(fields_autoplaced yes)
+		(property "Reference" "#PWR019"
+			(at 127 121.92 0)
+			(hide yes)
+			(show_name no)
+			(do_not_autoplace no)
+			(effects
+				(font
+					(size 1.27 1.27)
+				)
+			)
+		)
+		(property "Value" "GND"
+			(at 127 120.65 0)
+			(show_name no)
+			(do_not_autoplace no)
+			(effects
+				(font
+					(size 1.27 1.27)
+				)
+			)
+		)
+		(property "Footprint" ""
+			(at 127 115.57 0)
+			(hide yes)
+			(show_name no)
+			(do_not_autoplace no)
+			(effects
+				(font
+					(size 1.27 1.27)
+				)
+			)
+		)
+		(property "Datasheet" ""
+			(at 127 115.57 0)
+			(hide yes)
+			(show_name no)
+			(do_not_autoplace no)
+			(effects
+				(font
+					(size 1.27 1.27)
+				)
+			)
+		)
+		(property "Description" "Power symbol creates a global label with name \"GND\" , ground"
+			(at 127 115.57 0)
+			(hide yes)
+			(show_name no)
+			(do_not_autoplace no)
+			(effects
+				(font
+					(size 1.27 1.27)
+				)
+			)
+		)
+		(pin "1"
+		)
+		(instances
+			(project "SinglePhotonDetector"
+				(path "/74b1e2e4-bcd1-4fcc-9b31-cf62bc4f9919/434ab443-3fd9-4b87-8fcd-b0d2eb400dca"
+					(reference "#PWR019")
+					(unit 1)
+				)
+			)
 		)
 	)
@@
 			)
 		)
-		(property "Value" "JS202011JAQN"
+		(property "Value" "JS202011JCQN"
 			(at 168.148 80.772 0)
 			(show_name no)
@@
 					(unit 1)
 				)
+			)
+		)
+	)
+	(symbol
+		(lib_id "power:GND")
+		(at 157.48 115.57 0)
+		(unit 1)
+		(body_style 1)
+		(exclude_from_sim no)
+		(in_bom yes)
+		(on_board yes)
+		(in_pos_files yes)
+		(dnp no)
+		(fields_autoplaced yes)
+		(property "Reference" "#PWR020"
+			(at 157.48 121.92 0)
+			(hide yes)
+			(show_name no)
+			(do_not_autoplace no)
+			(effects
+				(font
+					(size 1.27 1.27)
+				)
+			)
+		)
+		(property "Value" "GND"
+			(at 157.48 120.65 0)
+			(show_name no)
+			(do_not_autoplace no)
+			(effects
+				(font
+					(size 1.27 1.27)
+				)
+			)
+		)
+		(property "Footprint" ""
+			(at 157.48 115.57 0)
+			(hide yes)
+			(show_name no)
+			(do_not_autoplace no)
+			(effects
+				(font
+					(size 1.27 1.27)
+				)
+			)
+		)
+		(property "Datasheet" ""
+			(at 157.48 115.57 0)
+			(hide yes)
+			(show_name no)
+			(do_not_autoplace no)
+			(effects
+				(font
+					(size 1.27 1.27)
+				)
+			)
+		)
+		(property "Description" "Power symbol creates a global label with name \"GND\" , ground"
+			(at 157.48 115.57 0)
+			(hide yes)
+			(show_name no)
+			(do_not_autoplace no)
+			(effects
+				(font
+					(size 1.27 1.27)
+				)
+			)
+		)
+		(pin "1"
+		)
+		(instances
+			(project "SinglePhotonDetector"
+				(path "/74b1e2e4-bcd1-4fcc-9b31-cf62bc4f9919/434ab443-3fd9-4b87-8fcd-b0d2eb400dca"
+					(reference "#PWR020")
+					(unit 1)
+				)
