File: 02_PCB/Fast_SiPM_Photodetector/Photodetector.kicad_sch (KiCad schematic)
At the start: 14 parts, among them IC3 MICROFC-30035-SMT-TR1, IC4 NCP731ADNADJR2G, Q2 MMBT6427LT1G

Commit message: feat(detector): update schematic and pcb after first prototype
Parts:
- C14: value 10n; 100V -> 10n;100V
- RV1: value 3314J-1-103 -> 3314J-1-102
Other:
- note added: "Photodetector"
- note added: "V_BIAS adjustable between 23.8 V ... 29.1 V with the selected resistor values"
- note removed: "V_BIAS adjustable between 28.8 V ... 29.1 V with the selected resistor values"
Changed lines of the file:
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@@
 		(title "Fast SiPM Photodetector")
 	)
-	(text "V_BIAS adjustable between\n28.8 V ... 29.1 V with the\nselected resistor values"
+	(text "V_BIAS adjustable between\n23.8 V ... 29.1 V with the\nselected resistor values"
 		(exclude_from_sim no)
 		(at 38.354 175.768 0)
@@
 			(font
 				(size 1.27 1.27)
+			)
+		)
+	)
+	(text "Photodetector"
+		(exclude_from_sim no)
+		(at 147.574 36.068 0)
+		(effects
+			(font
+				(size 3.81 3.81)
+				(thickness 0.508)
+				(bold yes)
 			)
 		)
@@
 		(shape input)
 		(at 55.88 57.15 180)
-		(effects
-			(font
-				(size 1.27 1.27)
-			)
-			(justify right)
-		)
-	)
-	(hierarchical_label "GND"
-		(shape input)
-		(at 81.28 87.63 270)
 		(effects
 			(font
@@
 			)
 		)
-		(property "Value" "10n; 100V"
+		(property "Value" "10n;100V"
 			(at 111.76 135.8899 0)
 			(show_name no)
@@
 	)
 	(symbol
+		(lib_id "power:GND")
+		(at 81.28 87.63 0)
+		(unit 1)
+		(body_style 1)
+		(exclude_from_sim no)
+		(in_bom yes)
+		(on_board yes)
+		(in_pos_files yes)
+		(dnp no)
+		(fields_autoplaced yes)
+		(property "Reference" "#PWR029"
+			(at 81.28 93.98 0)
+			(hide yes)
+			(show_name no)
+			(do_not_autoplace no)
+			(effects
+				(font
+					(size 1.27 1.27)
+				)
+			)
+		)
+		(property "Value" "GND"
+			(at 81.28 92.71 0)
+			(show_name no)
+			(do_not_autoplace no)
+			(effects
+				(font
+					(size 1.27 1.27)
+				)
+			)
+		)
+		(property "Footprint" ""
+			(at 81.28 87.63 0)
+			(hide yes)
+			(show_name no)
+			(do_not_autoplace no)
+			(effects
+				(font
+					(size 1.27 1.27)
+				)
+			)
+		)
+		(property "Datasheet" ""
+			(at 81.28 87.63 0)
+			(hide yes)
+			(show_name no)
+			(do_not_autoplace no)
+			(effects
+				(font
+					(size 1.27 1.27)
+				)
+			)
+		)
+		(property "Description" "Power symbol creates a global label with name \"GND\" , ground"
+			(at 81.28 87.63 0)
+			(hide yes)
+			(show_name no)
+			(do_not_autoplace no)
+			(effects
+				(font
+					(size 1.27 1.27)
+				)
+			)
+		)
+		(pin "1"
+		)
+		(instances
+			(project "SinglePhotonDetector"
+				(path "/74b1e2e4-bcd1-4fcc-9b31-cf62bc4f9919/4b98d106-56f1-476c-9227-b8a48a6c8e2a"
+					(reference "#PWR029")
+					(unit 1)
+				)
+			)
+		)
+	)
+	(symbol
 		(lib_id "CustomParts:NCP731ADNADJR2G")
 		(at 167.64 57.15 0)
@@
 			)
 		)
-		(property "Value" "3314J-1-103"
+		(property "Value" "3314J-1-102"
 			(at 196.85 88.9001 0)
 			(show_name no)
