File: 02_PCB/Fast_SiPM_Photodetector/TemperatureSensor.kicad_sch (KiCad schematic)
At the start: 7 parts, among them U2 TLV70033_SOT23-5, U3 MCP9700Ax-ETT

Commit message: feat(detector): update schematic and pcb after first prototype
Parts:
- U2: value TLV70033_SOT23-5 -> TLV70033DDCR
Other:
- note added: "Temperature Sensor"
- moved on the sheet: C23, C24, C25, C26, R18, U2, U3
