File: 02_PCB/Fast_SiPM_Photodetector/Amplifier.kicad_sch (KiCad schematic)
At the start: 10 parts, among them Q3 MMBT6427LT1G, U1 GALI-S66

Commit message: feat(detector): update schematic and pcb after first prototype
Parts:
- removed FB2: BLM18AG601SN1D, Inductor_SMD:L_0603_1608Metric, symbol Device:FerriteBead
- added L3: 1008CS-222XGRC, Inductor_SMD:L_1008_2520Metric, symbol Device:L
- added L4: 0603HP-R10XGRW, Inductor_SMD:L_0603_1608Metric, symbol Device:L
- C20, C22: value 10n -> 10nF;25V;C0G; footprint Capacitor_SMD:C_0603_1608Metric -> Capacitor_SMD:C_0402_1005Metric
- R17: value 1.5k;1% -> 169;1%; footprint Resistor_SMD:R_0603_1608Metric -> Resistor_SMD:R_0805_2012Metric
Connections:
- net at C22.1, U1.3: now also L4.2
- net at R17.1: now also L3.1
- new net: L3.2, L4.1
Other:
- note added: "Amplifier"
- note added: "For better performance use a Thin Film Resistor"
- note added: "Use high-frequency caps (C0G/NP0)"
- note removed: "For better performance choose a Thin Film Resistor (e.g. MELF)"
- note removed: "Use high-frequency C0G/NP0 or low-ESR X7R capacitors"
- moved on the sheet: C18, C19, C21, Q3, R16, R17

Commit message: chore: PCB V0.2 as ordered on 06.10.2026
Parts:
- added MP1, MP2, MP3, MP4, MP5, MP6: S0941-46R, CustomParts:S094146R, symbol CustomParts:S0941-46R
Connections:
- net GND: now also MP1.1, MP1.2, MP1.3, MP1.4, MP1.5, MP2.1, MP2.2, MP2.3, MP2.4, MP2.5, MP3.1, MP3.2, MP3.3, MP3.4, MP3.5, MP4.1, MP4.2, MP4.3, MP4.4, MP4.5, MP5.1, MP5.2, MP5.3, MP5.4, MP5.5, MP6.1, MP6.2, MP6.3, MP6.4, MP6.5
Other:
- note added: "Shielding Can Clips"
