File: 02_PCB/Fast_SiPM_Photodetector/Fast_SiPM_Photodetector.kicad_pcb (KiCad board)
At the start: 4 copper layers, 60 x 40 mm, 70 parts, among them IC1 LT8365JMSE, IC2 LMR51606XDBVR, IC3 MICROFC-30035-SMT-TR1, IC4 NCP731ADNADJR2G, J1 PTSM 0,5/ 2-HH-2,5-SMD R32, J2 SMA, J3 PTSM 0,5/ 4-HH-2,5-SMD R32, Q1 PJA3463_R1_00001, Q2 MMBT6427LT1G, Q3 MMBT6427LT1G, SW1 JS202011JAQN, U1 GALI-S66, U2 TLV70033_SOT23-5, U3 MCP9700Ax-ETT

Commit message: feat(detector): update schematic and pcb after first prototype
Parts:
- removed C8: 10u;50V, Capacitor_SMD:C_1206_3216Metric
- removed FB2: BLM18AG601SN1D, Inductor_SMD:L_0603_1608Metric
- added C27: 10u;50V, Capacitor_SMD:C_1206_3216Metric, F.Cu at (132.3, 84.9)
- added C28: 10u;50V, Capacitor_SMD:C_1206_3216Metric, F.Cu at (132.3, 88.7)
- added C29: 100n;100V, Capacitor_SMD:C_0603_1608Metric, F.Cu at (132.3, 90.6)
- added FB3: BLM18AG601SN1D, Inductor_SMD:L_0603_1608Metric, F.Cu at (132.4, 86.8)
- added L3: 1008CS-222XGRC, Inductor_SMD:L_1008_2520Metric, F.Cu at (169.2, 94.7)
- added L4: 0603HP-R10XGRW, Inductor_SMD:L_0603_1608Metric, F.Cu at (169.5, 98.0)
- C14: value 10n; 100V -> 10n;100V
- C20, C22: value 10n -> 10nF;25V;C0G; footprint Capacitor_SMD:C_0603_1608Metric -> Capacitor_SMD:C_0402_1005Metric
- D2: value SMD115PBQ-TP -> RB021VAM90TR
- IC2: value LMR51606XDBVR -> LMR51606XFDBVR
- L2: footprint Inductor_SMD:L_Wuerth_MAPI-5020 -> CustomParts:L_Wuerth_MAPI-5020-Custom
- R17: value 1.5k;1% -> 169;1%; footprint Resistor_SMD:R_0603_1608Metric -> Resistor_SMD:R_0805_2012Metric
- RV1: value 3314J-1-103 -> 3314J-1-102
- SW1: value JS202011JAQN -> JS202011JCQN
- U2: value TLV70033_SOT23-5 -> TLV70033DDCR
- moved C25 26.2 mm to (147.4, 105.5), turned to 90 degrees
- moved U3 22.4 mm to (150.0, 105.5)
- moved C26 18.7 mm to (152.6, 105.5), turned to -90 degrees
- moved R18 16.7 mm to (154.1, 105.5), turned to 90 degrees
- moved C19 16.4 mm to (166.6, 88.7)
- moved C18 16.3 mm to (160.1, 88.8)
- moved Q3 16.3 mm to (164.1, 88.2)
- moved R16 16.3 mm to (161.6, 88.8)
- moved R9 13.5 mm to (142.8, 90.3), turned to 180 degrees
- moved R17 11.3 mm to (165.5, 94.7), turned to 180 degrees
- moved C21 11.1 mm to (162.3, 94.7), turned to 180 degrees
- moved R10 9.86 mm to (139.8, 90.3), turned to 180 degrees
- moved C23 5.01 mm to (166.6, 84.0), turned to 90 degrees
- moved C24 4.31 mm to (160.8, 84.0), turned to 90 degrees
- moved R12 3.28 mm to (132.3, 83.0)
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Connections:
- net /Amplifier/VIN renamed /LVPowerSupply/LV_OUT
- net /HVPowerSupply/EN renamed /HVPowerSupply/HV_EN
- net /HVPowerSupply/FBX renamed /HVPowerSupply/HV_FB
- net Net-(IC2-EN) renamed /LVPowerSupply/LV_EN
- net Net-(IC2-FB) renamed /LVPowerSupply/LV_FB
- IC2 pad 5: /HVPowerSupply/VIN -> Net-(IC2-VIN)
Routing:
- net /TemperatureSensor/TEMP_OUT: track 46.1 -> 8.17 mm, vias 2 -> 0
- net Net-(U2-OUT): track 10.5 -> 37.5 mm, vias 0 -> 2
- net Net-(D1-K): track 2.10 -> 12.5 mm
- net Net-(IC2-VIN): track 0.00 -> 8.82 mm
- net /HVPowerSupply/VIN: track 31.4 -> 38.3 mm
- net /HVPowerSupply/HV_OUT: track 39.3 -> 32.5 mm
- net /LVPowerSupply/LV_OUT: track 52.0 -> 45.4 mm
- net GND: track 35.2 -> 31.0 mm, vias 193 -> 247
- net Net-(Q3-E): track 4.81 -> 8.75 mm
- net /LVPowerSupply/LV_FB: track 5.40 -> 8.13 mm
- net Net-(L3-Pad2): track 0.00 -> 2.73 mm
- net /LVPowerSupply/LV_EN: track 7.01 -> 9.12 mm
- net Net-(U3-V_{OUT}): track 3.38 -> 4.24 mm
- net /Photodetector/BIAS_ADJ: track 59.4 -> 60.1 mm
- net Net-(L3-Pad1): track 1.39 -> 2.04 mm
- removed copper zone on In2.Cu, net /HVPowerSupply/VIN
- removed copper zone on In2.Cu, net Net-(D1-K)
Other:
- outline, holes or cut-outs redrawn

Commit message: chore: PCB V0.2 as ordered on 06.10.2026
Parts:
- added MP1: S0941-46R, CustomParts:S094146R, F.Cu at (168.5, 95.0)
- added MP2: S0941-46R, CustomParts:S094146R, F.Cu at (159.5, 95.0)
- added MP3: S0941-46R, CustomParts:S094146R, F.Cu at (156.5, 100.0)
- added MP4: S0941-46R, CustomParts:S094146R, F.Cu at (159.5, 105.0)
- added MP5: S0941-46R, CustomParts:S094146R, F.Cu at (168.6, 105.0)
- added MP6: S0941-46R, CustomParts:S094146R, F.Cu at (171.5, 100.0)
- moved C18 3.52 mm to (158.8, 92.0)
- moved C19 3.52 mm to (165.2, 92.0)
- moved Q3 3.52 mm to (162.8, 91.5)
- moved R16 3.52 mm to (160.2, 92.0)
- moved C20 3.26 mm to (159.5, 102.9)
- moved C22 3.26 mm to (168.5, 102.9)
- moved L4 3.26 mm to (168.0, 100.9)
- moved U1 3.26 mm to (164.0, 100.9)
- moved L3 3.18 mm to (167.7, 97.5)
- moved C21 2.83 mm to (160.8, 97.1)
- moved R17 2.83 mm to (164.0, 97.1)
- moved C23 1.93 mm to (165.3, 85.5)
- moved C24 1.93 mm to (159.5, 85.5)
- moved U2 1.93 mm to (162.5, 85.5)
- moved C25 0.60 mm to (146.8, 105.5)
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Routing:
- net /LVPowerSupply/LV_OUT: track 45.4 -> 48.9 mm, vias 8 -> 9
- net Net-(U2-OUT): track 37.5 -> 34.5 mm
- net GND: track 31.0 -> 33.0 mm, vias 247 -> 264
- net /Amplifier/SIG_IN: track 9.35 -> 7.37 mm
- net /Amplifier/SIG_OUT: track 7.06 -> 8.99 mm
- net /HVPowerSupply/VIN: track 38.3 -> 37.0 mm
- net Net-(U3-V_{OUT}): track 4.24 -> 3.32 mm
- net Net-(Q3-E): track 8.75 -> 8.20 mm
- net /LVPowerSupply/LV_FB: track 8.13 -> 7.60 mm
Other:
- board text added: "Hannes Duske 10.2026 V0.2"
- board text removed: "Hannes Duske 09.2026 V0.1"
